Commit message: configure base_link origin

File: sayebot_description/urdf/sayebot.urdf.xacro (robot description, xacro)
@@ -7,5 +7,5 @@
                 <mesh filename="package://sayebot_description/meshes/BaseReduced.dae"/>
             </geometry>
-            <origin xyz="0 0 0" rpy="0 0 0"/>
+            <origin xyz="0 -0.1371 0.0115" rpy="0 0 0"/>
         </visual>
     </link>

Commit message: add the rest of links and joints

File: sayebot_description/urdf/sayebot.urdf.xacro (robot description, xacro)
@@ -7,5 +7,5 @@
                 <mesh filename="package://sayebot_description/meshes/BaseReduced.dae"/>
             </geometry>
-            <origin xyz="0 -0.1371 0.0115" rpy="0 0 0"/>
+            <origin xyz="0.1371 0 0" rpy="0 0 ${pi/2}"/>
         </visual>
     </link>
@@ -13,5 +13,70 @@
         <parent link="base_footprint"/>
         <child link="base_link"/>
+        <origin xyz="0 0 0.0115" rpy="0 0 0"/>
+    </joint>
+    <link name="upper_link">
+        <visual>
+                <geometry>
+                        <mesh filename="package://sayebot_description/meshes/TopReduced.dae"/>
+                </geometry>
+                <origin xyz="0.1371 0 0" rpy="0 0 ${pi/2}"/>
+        </visual>
+    </link>
+    <joint name="upper_joint" type="fixed">
+        <parent link="base_link"/>
+        <child link="upper_link"/>
         <origin xyz="0 0 0" rpy="0 0 0"/>
     </joint>
+    <link name="right_forward_wheel_link">
+        <visual>
+                <geometry>
+                        <mesh filename="package://sayebot_description/meshes/Wheel.dae"/>
+                </geometry>
+                <origin xyz="0 0 0" rpy="0 0 0"/>
+        </visual>
+    </link>
+    <joint name="right_forward_wheel_joint" type="fixed">
+        <parent link="base_link"/>
+        <child link="right_forward_wheel_link"/>
+        <origin xyz="0.11 -0.1 0.0115" rpy="0 0 0"/>
+    </joint>
+    <link name="right_backward_wheel_link">
+        <visual>
+                <geometry>
+                        <mesh filename="package://sayebot_description/meshes/Wheel.dae"/>
+                </geometry>
+                <origin xyz="0 0 0" rpy="0 0 0"/>
+        </visual>
+    </link>
+    <joint name="right_backward_wheel_joint" type="fixed">
+        <parent link="base_link"/>
+        <child link="right_backward_wheel_link"/>
+        <origin xyz="-0.115 -0.1 0.0115" rpy="0 0 0"/>
+    </joint>
+    <link name="left_forward_wheel_link">
+        <visual>
+                <geometry>
+                        <mesh filename="package://sayebot_description/meshes/Wheel.dae"/>
+                </geometry>
+                <origin xyz="0 0 0" rpy="0 0 ${pi}"/>
+        </visual>
+    </link>
+    <joint name="left_forward_wheel_joint" type="fixed">
+        <parent link="base_link"/>
+        <child link="left_forward_wheel_link"/>
+        <origin xyz="0.11 0.1 0.0115" rpy="0 0 0"/>
+    </joint>
+    <link name="left_backward_wheel_link">
+        <visual>
+                <geometry>
+                        <mesh filename="package://sayebot_description/meshes/Wheel.dae"/>
+                </geometry>
+                <origin xyz="0 0 0" rpy="0 0 ${pi}"/>
+        </visual>
+    </link>
+    <joint name="left_backward_wheel_joint" type="fixed">
+        <parent link="base_link"/>
+        <child link="left_backward_wheel_link"/>
+        <origin xyz="-0.115 0.1 0.0115" rpy="0 0 0"/>
+    </joint>
 </robot>

Commit message: fix wheel displacement

File: sayebot_description/urdf/sayebot.urdf.xacro (robot description, xacro)
@@ -33,5 +33,5 @@
                         <mesh filename="package://sayebot_description/meshes/Wheel.dae"/>
                 </geometry>
-                <origin xyz="0 0 0" rpy="0 0 0"/>
+                <origin xyz="0 -0.015 0" rpy="0 0 0"/>
         </visual>
     </link>
@@ -39,5 +39,5 @@
         <parent link="base_link"/>
         <child link="right_forward_wheel_link"/>
-        <origin xyz="0.11 -0.1 0.0115" rpy="0 0 0"/>
+        <origin xyz="0.11 -0.09 0.0115" rpy="0 0 0"/>
     </joint>
     <link name="right_backward_wheel_link">
@@ -46,5 +46,5 @@
                         <mesh filename="package://sayebot_description/meshes/Wheel.dae"/>
                 </geometry>
-                <origin xyz="0 0 0" rpy="0 0 0"/>
+                <origin xyz="0 -0.015 0" rpy="0 0 0"/>
         </visual>
     </link>
@@ -52,5 +52,5 @@
         <parent link="base_link"/>
         <child link="right_backward_wheel_link"/>
-        <origin xyz="-0.115 -0.1 0.0115" rpy="0 0 0"/>
+        <origin xyz="-0.115 -0.09 0.0115" rpy="0 0 0"/>
     </joint>
     <link name="left_forward_wheel_link">
@@ -59,5 +59,5 @@
                         <mesh filename="package://sayebot_description/meshes/Wheel.dae"/>
                 </geometry>
-                <origin xyz="0 0 0" rpy="0 0 ${pi}"/>
+                <origin xyz="0 0.015 0" rpy="0 0 ${pi}"/>
         </visual>
     </link>
@@ -65,5 +65,5 @@
         <parent link="base_link"/>
         <child link="left_forward_wheel_link"/>
-        <origin xyz="0.11 0.1 0.0115" rpy="0 0 0"/>
+        <origin xyz="0.11 0.09 0.0115" rpy="0 0 0"/>
     </joint>
     <link name="left_backward_wheel_link">
@@ -72,5 +72,5 @@
                         <mesh filename="package://sayebot_description/meshes/Wheel.dae"/>
                 </geometry>
-                <origin xyz="0 0 0" rpy="0 0 ${pi}"/>
+                <origin xyz="0 0.015 0" rpy="0 0 ${pi}"/>
         </visual>
     </link>
@@ -78,5 +78,5 @@
         <parent link="base_link"/>
         <child link="left_backward_wheel_link"/>
-        <origin xyz="-0.115 0.1 0.0115" rpy="0 0 0"/>
+        <origin xyz="-0.115 0.09 0.0115" rpy="0 0 0"/>
     </joint>
 </robot>

Commit message: add collision to wheel

File: sayebot_description/urdf/sayebot.urdf.xacro (robot description, xacro)
@@ -35,9 +35,17 @@
                 <origin xyz="0 -0.015 0" rpy="0 0 0"/>
         </visual>
+        <collision>
+            <geometry>
+                <cylinder radius="0.0365" length="0.03"/>
+            </geometry>
+            <origin xyz="0 0 0" rpy="${pi/2} 0 0"/>
+        </collision>
     </link>
-    <joint name="right_forward_wheel_joint" type="fixed">
+    <joint name="right_forward_wheel_joint" type="revolute">
         <parent link="base_link"/>
         <child link="right_forward_wheel_link"/>
         <origin xyz="0.11 -0.09 0.0115" rpy="0 0 0"/>
+        <axis xyz="0 0 1"/>
+        <limit effort="5" lower="-0.5" upper="0.5" velocity="1.0"/>
     </joint>
     <link name="right_backward_wheel_link">
@@ -48,9 +56,16 @@
                 <origin xyz="0 -0.015 0" rpy="0 0 0"/>
         </visual>
+        <collision>
+            <geometry>
+                <cylinder radius="0.0365" length="0.03"/>
+            </geometry>
+            <origin xyz="0 0 0" rpy="${pi/2} 0 0"/>
+        </collision>
     </link>
-    <joint name="right_backward_wheel_joint" type="fixed">
+    <joint name="right_backward_wheel_joint" type="continuous">
         <parent link="base_link"/>
         <child link="right_backward_wheel_link"/>
         <origin xyz="-0.115 -0.09 0.0115" rpy="0 0 0"/>
+        <axis xyz="0 1 0"/>
     </joint>
     <link name="left_forward_wheel_link">
@@ -61,9 +76,17 @@
                 <origin xyz="0 0.015 0" rpy="0 0 ${pi}"/>
         </visual>
+        <collision>
+            <geometry>
+                <cylinder radius="0.0365" length="0.03"/>
+            </geometry>
+            <origin xyz="0 0 0" rpy="${pi/2} 0 0"/>
+        </collision>
     </link>
-    <joint name="left_forward_wheel_joint" type="fixed">
+    <joint name="left_forward_wheel_joint" type="revolute">
         <parent link="base_link"/>
         <child link="left_forward_wheel_link"/>
         <origin xyz="0.11 0.09 0.0115" rpy="0 0 0"/>
+        <axis xyz="0 0 1"/>
+        <limit effort="5" lower="-0.5" upper="0.5" velocity="1.0"/>
     </joint>
     <link name="left_backward_wheel_link">
@@ -74,9 +97,16 @@
                 <origin xyz="0 0.015 0" rpy="0 0 ${pi}"/>
         </visual>
+        <collision>
+            <geometry>
+                <cylinder radius="0.0365" length="0.03"/>
+            </geometry>
+            <origin xyz="0 0 0" rpy="${pi/2} 0 0"/>
+        </collision>
     </link>
-    <joint name="left_backward_wheel_joint" type="fixed">
+    <joint name="left_backward_wheel_joint" type="continuous">
         <parent link="base_link"/>
         <child link="left_backward_wheel_link"/>
         <origin xyz="-0.115 0.09 0.0115" rpy="0 0 0"/>
+        <axis xyz="0 1 0"/>
     </joint>
 </robot>

Commit message: add the rest of the collision

File: sayebot_description/urdf/sayebot.urdf.xacro (robot description, xacro)
@@ -9,4 +9,16 @@
             <origin xyz="0.1371 0 0" rpy="0 0 ${pi/2}"/>
         </visual>
+        <visual>
+            <geometry>
+                    <mesh filename="package://sayebot_description/meshes/TopReduced.dae"/>
+            </geometry>
+            <origin xyz="0.1371 0 0" rpy="0 0 ${pi/2}"/>
+        </visual>
+        <collision>
+            <geometry>
+                <box size="0.3 0.09 0.12"/>
+            </geometry>
+            <origin xyz="-0.03 0 0.05" rpy="-${pi/2} 0 0"/>
+        </collision>
     </link>
     <joint name="base_joint" type="fixed">
@@ -14,17 +26,4 @@
         <child link="base_link"/>
         <origin xyz="0 0 0.0115" rpy="0 0 0"/>
-    </joint>
-    <link name="upper_link">
-        <visual>
-                <geometry>
-                        <mesh filename="package://sayebot_description/meshes/TopReduced.dae"/>
-                </geometry>
-                <origin xyz="0.1371 0 0" rpy="0 0 ${pi/2}"/>
-        </visual>
-    </link>
-    <joint name="upper_joint" type="fixed">
-        <parent link="base_link"/>
-        <child link="upper_link"/>
-        <origin xyz="0 0 0" rpy="0 0 0"/>
     </joint>
     <link name="right_forward_wheel_link">

Commit message: add the inertial

File: sayebot_description/urdf/sayebot.urdf.xacro (robot description, xacro)
@@ -3,4 +3,11 @@
     <link name="base_footprint"/>
     <link name="base_link">
+        <inertial>
+            <mass value="3.0" />
+            <inertia ixx="0.0054" ixy="0.0"     ixz="0.0"
+                                    iyy="0.0252" iyz="0.0"
+                                                    izz="0.0252" />
+            <origin xyz="0.0 0.0 0.038" rpy="0.0 0.0 0.0" />
+        </inertial>
         <visual>
             <geometry>
@@ -19,5 +26,5 @@
                 <box size="0.3 0.09 0.12"/>
             </geometry>
-            <origin xyz="-0.03 0 0.05" rpy="-${pi/2} 0 0"/>
+            <origin xyz="-0.03 0 0.06" rpy="0 0 0"/>
         </collision>
     </link>
@@ -28,9 +35,16 @@
     </joint>
     <link name="right_forward_wheel_link">
+        <inertial>
+            <mass value="0.05" />
+            <inertia ixx="0.00003331" ixy="0.0"     ixz="0.0"
+                                    iyy="0.0000204" iyz="0.0"
+                                                    izz="0.0000204" />
+            <origin xyz="0.0 0.0 0.0" rpy="0.0 0.0 0.0" />
+        </inertial>
         <visual>
-                <geometry>
-                        <mesh filename="package://sayebot_description/meshes/Wheel.dae"/>
-                </geometry>
-                <origin xyz="0 -0.015 0" rpy="0 0 0"/>
+            <geometry>
+                <mesh filename="package://sayebot_description/meshes/Wheel.dae"/>
+            </geometry>
+            <origin xyz="0 -0.015 0" rpy="0 0 0"/>
         </visual>
         <collision>
@@ -49,9 +63,16 @@
     </joint>
     <link name="right_backward_wheel_link">
+        <inertial>
+            <mass value="0.05" />
+            <inertia ixx="0.00003331" ixy="0.0"     ixz="0.0"
+                                    iyy="0.0000204" iyz="0.0"
+                                                    izz="0.0000204" />
+            <origin xyz="0.0 0.0 0.0" rpy="0.0 0.0 0.0" />
+        </inertial>
         <visual>
-                <geometry>
-                        <mesh filename="package://sayebot_description/meshes/Wheel.dae"/>
-                </geometry>
-                <origin xyz="0 -0.015 0" rpy="0 0 0"/>
+            <geometry>
+                <mesh filename="package://sayebot_description/meshes/Wheel.dae"/>
+            </geometry>
+            <origin xyz="0 -0.015 0" rpy="0 0 0"/>
         </visual>
         <collision>
@@ -69,9 +90,16 @@
     </joint>
     <link name="left_forward_wheel_link">
+        <inertial>
+            <mass value="0.05" />
+            <inertia ixx="0.00003331" ixy="0.0"     ixz="0.0"
+                                    iyy="0.0000204" iyz="0.0"
+                                                    izz="0.0000204" />
+            <origin xyz="0.0 0.0 0.0" rpy="0.0 0.0 0.0" />
+        </inertial>
         <visual>
-                <geometry>
-                        <mesh filename="package://sayebot_description/meshes/Wheel.dae"/>
-                </geometry>
-                <origin xyz="0 0.015 0" rpy="0 0 ${pi}"/>
+            <geometry>
+                <mesh filename="package://sayebot_description/meshes/Wheel.dae"/>
+            </geometry>
+            <origin xyz="0 0.015 0" rpy="0 0 ${pi}"/>
         </visual>
         <collision>
@@ -90,9 +118,16 @@
     </joint>
     <link name="left_backward_wheel_link">
+        <inertial>
+            <mass value="0.05" />
+            <inertia ixx="0.00003331" ixy="0.0"     ixz="0.0"
+                                    iyy="0.0000204" iyz="0.0"
+                                                    izz="0.0000204" />
+            <origin xyz="0.0 0.0 0.0" rpy="0.0 0.0 0.0" />
+        </inertial>
         <visual>
-                <geometry>
-                        <mesh filename="package://sayebot_description/meshes/Wheel.dae"/>
-                </geometry>
-                <origin xyz="0 0.015 0" rpy="0 0 ${pi}"/>
+            <geometry>
+                <mesh filename="package://sayebot_description/meshes/Wheel.dae"/>
+            </geometry>
+            <origin xyz="0 0.015 0" rpy="0 0 ${pi}"/>
         </visual>
         <collision>

Commit message: add two more joint for steering the front wheels

File: sayebot_description/urdf/sayebot.urdf.xacro (robot description, xacro)
@@ -56,10 +56,17 @@
         </collision>
     </link>
-    <joint name="right_forward_wheel_joint" type="revolute">
+    <link name="right_forward_steer_link"/>
+    <joint name="right_forward_steer_joint" type="revolute">
         <parent link="base_link"/>
-        <child link="right_forward_wheel_link"/>
+        <child link="right_forward_steer_link"/>
         <origin xyz="0.11 -0.09 0.0115" rpy="0 0 0"/>
         <axis xyz="0 0 1"/>
         <limit effort="5" lower="-0.5" upper="0.5" velocity="1.0"/>
+    </joint>
+    <joint name="right_forward_wheel_joint" type="continuous">
+        <parent link="right_forward_steer_link"/>
+        <child link="right_forward_wheel_link"/>
+        <origin xyz="0 0 0" rpy="0 0 0"/>
+        <axis xyz="0 1 0"/>
     </joint>
     <link name="right_backward_wheel_link">
@@ -111,10 +118,17 @@
         </collision>
     </link>
-    <joint name="left_forward_wheel_joint" type="revolute">
+    <link name="left_forward_steer_link"/>
+    <joint name="left_forward_steer_joint" type="revolute">
         <parent link="base_link"/>
-        <child link="left_forward_wheel_link"/>
+        <child link="left_forward_steer_link"/>
         <origin xyz="0.11 0.09 0.0115" rpy="0 0 0"/>
         <axis xyz="0 0 1"/>
         <limit effort="5" lower="-0.5" upper="0.5" velocity="1.0"/>
+    </joint>
+    <joint name="left_forward_wheel_joint" type="continuous">
+        <parent link="left_forward_steer_link"/>
+        <child link="left_forward_wheel_link"/>
+        <origin xyz="0 0 0" rpy="0 0 0"/>
+        <axis xyz="0 1 0"/>
     </joint>
     <link name="left_backward_wheel_link">

Commit message: finish ackermann controller

File: sayebot_description/urdf/sayebot.urdf.xacro (robot description, xacro)
@@ -57,5 +57,13 @@
         </collision>
     </link>
-    <link name="right_forward_steer_link"/>
+    <link name="right_forward_steer_link">
+        <inertial>
+            <mass value="0.05" />
+            <inertia ixx="0.00003331" ixy="0.0"     ixz="0.0"
+                                    iyy="0.0000204" iyz="0.0"
+                                                    izz="0.0000204" />
+            <origin xyz="0.0 0.0 0.0" rpy="0.0 0.0 0.0" />
+        </inertial>
+    </link>
     <joint name="right_forward_steer_joint" type="revolute">
         <parent link="base_link"/>
@@ -119,5 +127,13 @@
         </collision>
     </link>
-    <link name="left_forward_steer_link"/>
+    <link name="left_forward_steer_link">
+        <inertial>
+            <mass value="0.05" />
+            <inertia ixx="0.00003331" ixy="0.0"     ixz="0.0"
+                                    iyy="0.0000204" iyz="0.0"
+                                                    izz="0.0000204" />
+            <origin xyz="0.0 0.0 0.0" rpy="0.0 0.0 0.0" />
+        </inertial>
+    </link>
     <joint name="left_forward_steer_joint" type="revolute">
         <parent link="base_link"/>

File: sayebot_description/urdf/sayebot_gazebo.xacro (robot description, xacro)
@@ -2,38 +2,26 @@
 <robot name="sayebot" xmlns:xacro="http://www.ros.org/wiki/xacro">
     <gazebo reference="left_forward_wheel_link">
-        <mu1>1000.0</mu1>
-        <mu2>1000.0</mu2>
-        <kp>100.0</kp>
-        <kd>10.0</kd>
-        <minDepth>0.001</minDepth>
-        <maxVel>0.1</maxVel>
-        <fdir1>1 0 0</fdir1>
+        <mu1>10.0</mu1>
+        <mu2>8.0</mu2>
+        <kp>10000000.0</kp>
+        <kd>1.0</kd>
     </gazebo>
     <gazebo reference="right_forward_wheel_link">
-        <mu1>1000.0</mu1>
-        <mu2>1000.0</mu2>
-        <kp>100.0</kp>
-        <kd>10.0</kd>
-        <minDepth>0.001</minDepth>
-        <maxVel>0.1</maxVel>
-        <fdir1>1 0 0</fdir1>
+        <mu1>10.0</mu1>
+        <mu2>8.0</mu2>
+        <kp>10000000.0</kp>
+        <kd>1.0</kd>
     </gazebo>
     <gazebo reference="left_backward_wheel_link">
-        <mu1>1000.0</mu1>
-        <mu2>1000.0</mu2>
-        <kp>100.0</kp>
-        <kd>10.0</kd>
-        <minDepth>0.001</minDepth>
-        <maxVel>0.1</maxVel>
-        <fdir1>1 0 0</fdir1>
+        <mu1>10.0</mu1>
+        <mu2>8.0</mu2>
+        <kp>10000000.0</kp>
+        <kd>1.0</kd>
     </gazebo>
     <gazebo reference="right_backward_wheel_link">
-        <mu1>1000.0</mu1>
-        <mu2>1000.0</mu2>
-        <kp>100.0</kp>
-        <kd>10.0</kd>
-        <minDepth>0.001</minDepth>
-        <maxVel>0.1</maxVel>
-        <fdir1>1 0 0</fdir1>
+        <mu1>10.0</mu1>
+        <mu2>8.0</mu2>
+        <kp>10000000.0</kp>
+        <kd>1.0</kd>
     </gazebo>
     <gazebo>

File: sayebot_description/urdf/sayebot_ros2_control.xacro (robot description, xacro)
@@ -6,10 +6,8 @@
         </hardware>
         <joint name="right_forward_wheel_joint">
-            <command_interface name="velocity"/>
             <state_interface name="position"/>
             <state_interface name="velocity"/>
         </joint>
         <joint name="left_forward_wheel_joint">
-            <command_interface name="velocity"/>
             <state_interface name="position"/>
             <state_interface name="velocity"/>

Commit message: add lidar link

File: sayebot_description/urdf/sayebot.urdf.xacro (robot description, xacro)
@@ -176,3 +176,16 @@
         <axis xyz="0 1 0"/>
     </joint>
+    <link name="laser_link">
+        <visual>
+            <geometry>
+                <mesh filename="package://sayebot_description/meshes/STL27L.dae"/>
+            </geometry>
+            <origin xyz="0 0 0.13" rpy="0 0 ${pi}"/>
+        </visual>
+    </link>
+    <joint name="laser_joint" type="fixed">
+        <parent link="base_link"/>
+        <child link="laser_link"/>
+        <origin xyz="0 0 0" rpy="0 0 0"/>
+    </joint>
 </robot>

Commit message: add laser scan gazebo plugin

File: sayebot_description/urdf/sayebot.urdf.xacro (robot description, xacro)
@@ -181,5 +181,5 @@
                 <mesh filename="package://sayebot_description/meshes/STL27L.dae"/>
             </geometry>
-            <origin xyz="0 0 0.13" rpy="0 0 ${pi}"/>
+            <origin xyz="0 0 -0.09" rpy="0 0 ${pi}"/>
         </visual>
     </link>
@@ -187,5 +187,5 @@
         <parent link="base_link"/>
         <child link="laser_link"/>
-        <origin xyz="0 0 0" rpy="0 0 0"/>
+        <origin xyz="0 0 0.22" rpy="0 0 0"/>
     </joint>
 </robot>

File: sayebot_description/urdf/sayebot_gazebo.xacro (robot description, xacro)
@@ -29,4 +29,36 @@
             <parameters>$(find sayebot_controller)/config/ackermann_controller.yaml</parameters>
         </plugin>
+        <plugin filename="ignition-gazebo-sensors-system" name="ignition::gazebo::systems::Sensors">
+            <render_engine>ogre2</render_engine>
+        </plugin>
+    </gazebo>
+    <gazebo reference="laser_link">
+        <sensor name="lidar" type="gpu_ray">
+            <always_on>true</always_on>
+            <visualize>true</visualize>
+            <topic>scan</topic>
+            <update_rate>5</update_rate>
+            <gz_frame_id>laser_link</gz_frame_id>
+            <lidar>
+                <scan>
+                    <horizontal>
+                        <samples>360</samples>
+                        <resolution>1.0</resolution>
+                        <min_angle>0.0</min_angle>
+                        <max_angle>6.28</max_angle>
+                    </horizontal>
+                </scan>
+                <range>
+                    <min>0.12</min>
+                    <max>12.0</max>
+                    <resolution>0.02</resolution>
+                </range>
+                <noise>
+                    <type>gaussion</type>
+                    <mean>0.0</mean>
+                    <stddev>0.01</stddev>
+                </noise>
+            </lidar>
+        </sensor>
     </gazebo>
 </robot>
