Commit message: add camera to the robot

File: sayebot_description/urdf/sayebot.urdf.xacro (robot description, xacro)
@@ -189,3 +189,19 @@
         <origin xyz="0 0 0.22" rpy="0 0 0"/>
     </joint>
+    <link name="camera_link">
+        <visual>
+            <geometry>
+                <mesh filename="package://sayebot_description/meshes/camera.STL" scale="0.5 0.5 0.5"/>
+            </geometry>
+            <origin xyz="0 0 0" rpy="0 0 0"/>
+        <material name="dark">
+            <color rgba="0.8 0.8 0.8 1"></color>
+        </material>
+        </visual>
+    </link>
+    <joint name="camera_joint" type="fixed">
+        <parent link="base_link"/>
+        <child link="camera_link"/>
+        <origin xyz="0.09 0 0.1" rpy="0 0 0"/>
+    </joint>
 </robot>

File: sayebot_description/urdf/sayebot_gazebo.xacro (robot description, xacro)
@@ -62,3 +62,23 @@
         </sensor>
     </gazebo>
+     <gazebo reference="camera_link">
+        <sensor name="camera" type="camera">
+            <always_on>true</always_on>
+            <update_rate>20</update_rate>
+            <visualize>true</visualize>
+            <topic>camera</topic>
+            <camera>
+                <horizontal_fov>1.5</horizontal_fov>
+                <image>
+                    <format>R8G8B8</format>
+                    <width>640</width>
+                    <height>480</height>
+                </image>
+                <clip>
+                    <near>0.1</near>
+                    <far>100</far>
+                </clip>
+            </camera>
+        </sensor>
+    </gazebo>
 </robot>

Commit message: resize the robo

File: sayebot_description/urdf/sayebot.urdf.xacro (robot description, xacro)
@@ -14,19 +14,19 @@
         <visual>
             <geometry>
-                <mesh filename="package://sayebot_description/meshes/BaseReduced.dae"/>
-            </geometry>
-            <origin xyz="0.1371 0 0" rpy="0 0 ${pi/2}"/>
-        </visual>
-        <visual>
-            <geometry>
-                    <mesh filename="package://sayebot_description/meshes/TopReduced.dae"/>
-            </geometry>
-            <origin xyz="0.1371 0 0" rpy="0 0 ${pi/2}"/>
-        </visual>
-        <collision>
-            <geometry>
-                <box size="0.3 0.09 0.12"/>
-            </geometry>
-            <origin xyz="-0.03 0 0.06" rpy="0 0 0"/>
+                <mesh filename="package://sayebot_description/meshes/BaseReduced.dae" scale="5 5 5"/>
+            </geometry>
+            <origin xyz="0.6855 0 0" rpy="0 0 ${pi/2}"/>
+        </visual>
+        <visual>
+            <geometry>
+                    <mesh filename="package://sayebot_description/meshes/TopReduced.dae" scale="5 5 5"/>
+            </geometry>
+            <origin xyz="0.6855 0 0" rpy="0 0 ${pi/2}"/>
+        </visual>
+        <collision>
+            <geometry>
+                <box size="1.5 0.45 0.6"/>
+            </geometry>
+            <origin xyz="-0.15 0 0.3" rpy="0 0 0"/>
         </collision>
     </link>
@@ -34,5 +34,5 @@
         <parent link="base_footprint"/>
         <child link="base_link"/>
-        <origin xyz="0 0 0.0115" rpy="0 0 0"/>
+        <origin xyz="0 0 0.0575" rpy="0 0 0"/>
     </joint>
     <link name="right_forward_wheel_link">
@@ -46,11 +46,11 @@
         <visual>
             <geometry>
-                <mesh filename="package://sayebot_description/meshes/Wheel.dae"/>
-            </geometry>
-            <origin xyz="0 -0.015 0" rpy="0 0 0"/>
-        </visual>
-        <collision>
-            <geometry>
-                <cylinder radius="0.0365" length="0.03"/>
+                <mesh filename="package://sayebot_description/meshes/Wheel.dae" scale="5 5 5"/>
+            </geometry>
+            <origin xyz="0 -0.075 0" rpy="0 0 0"/>
+        </visual>
+        <collision>
+            <geometry>
+                <cylinder radius="0.1825" length="0.15"/>
             </geometry>
             <origin xyz="0 0 0" rpy="${pi/2} 0 0"/>
@@ -69,5 +69,5 @@
         <parent link="base_link"/>
         <child link="right_forward_steer_link"/>
-        <origin xyz="0.11 -0.09 0.0115" rpy="0 0 0"/>
+        <origin xyz="0.55 -0.45 0.0575" rpy="0 0 0"/>
         <axis xyz="0 0 1"/>
         <limit effort="5" lower="-0.5" upper="0.5" velocity="1.0"/>
@@ -89,11 +89,11 @@
         <visual>
             <geometry>
-                <mesh filename="package://sayebot_description/meshes/Wheel.dae"/>
-            </geometry>
-            <origin xyz="0 -0.015 0" rpy="0 0 0"/>
-        </visual>
-        <collision>
-            <geometry>
-                <cylinder radius="0.0365" length="0.03"/>
+                <mesh filename="package://sayebot_description/meshes/Wheel.dae" scale="5 5 5"/>
+            </geometry>
+            <origin xyz="0 -0.075 0" rpy="0 0 0"/>
+        </visual>
+        <collision>
+            <geometry>
+                <cylinder radius="0.1825" length="0.15"/>
             </geometry>
             <origin xyz="0 0 0" rpy="${pi/2} 0 0"/>
@@ -103,5 +103,5 @@
         <parent link="base_link"/>
         <child link="right_backward_wheel_link"/>
-        <origin xyz="-0.115 -0.09 0.0115" rpy="0 0 0"/>
+        <origin xyz="-0.575 -0.45 0.0575" rpy="0 0 0"/>
         <axis xyz="0 1 0"/>
     </joint>
@@ -116,11 +116,11 @@
         <visual>
             <geometry>
-                <mesh filename="package://sayebot_description/meshes/Wheel.dae"/>
-            </geometry>
-            <origin xyz="0 0.015 0" rpy="0 0 ${pi}"/>
-        </visual>
-        <collision>
-            <geometry>
-                <cylinder radius="0.0365" length="0.03"/>
+                <mesh filename="package://sayebot_description/meshes/Wheel.dae" scale="5 5 5"/>
+            </geometry>
+            <origin xyz="0 0.075 0" rpy="0 0 ${pi}"/>
+        </visual>
+        <collision>
+            <geometry>
+                <cylinder radius="0.1825" length="0.15"/>
             </geometry>
             <origin xyz="0 0 0" rpy="${pi/2} 0 0"/>
@@ -139,5 +139,5 @@
         <parent link="base_link"/>
         <child link="left_forward_steer_link"/>
-        <origin xyz="0.11 0.09 0.0115" rpy="0 0 0"/>
+        <origin xyz="0.55 0.45 0.0575" rpy="0 0 0"/>
         <axis xyz="0 0 1"/>
         <limit effort="5" lower="-0.5" upper="0.5" velocity="1.0"/>
@@ -159,11 +159,11 @@
         <visual>
             <geometry>
-                <mesh filename="package://sayebot_description/meshes/Wheel.dae"/>
-            </geometry>
-            <origin xyz="0 0.015 0" rpy="0 0 ${pi}"/>
-        </visual>
-        <collision>
-            <geometry>
-                <cylinder radius="0.0365" length="0.03"/>
+                <mesh filename="package://sayebot_description/meshes/Wheel.dae" scale="5 5 5"/>
+            </geometry>
+            <origin xyz="0 0.075 0" rpy="0 0 ${pi}"/>
+        </visual>
+        <collision>
+            <geometry>
+                <cylinder radius="0.1825" length="0.15"/>
             </geometry>
             <origin xyz="0 0 0" rpy="${pi/2} 0 0"/>
@@ -173,11 +173,11 @@
         <parent link="base_link"/>
         <child link="left_backward_wheel_link"/>
-        <origin xyz="-0.115 0.09 0.0115" rpy="0 0 0"/>
-        <axis xyz="0 1 0"/>
-    </joint>
-    <link name="laser_link">
-        <visual>
-            <geometry>
-                <mesh filename="package://sayebot_description/meshes/STL27L.dae"/>
+        <origin xyz="-0.575 0.45 0.0575" rpy="0 0 0"/>
+        <axis xyz="0 1 0"/>
+    </joint>
+    <!-- <link name="laser_link">
+        <visual>
+            <geometry>
+                <mesh filename="package://sayebot_description/meshes/STL27L.dae" scale="5 5 5"/>
             </geometry>
             <origin xyz="0 0 -0.09" rpy="0 0 ${pi}"/>
@@ -188,11 +188,11 @@
         <child link="laser_link"/>
         <origin xyz="0 0 0.22" rpy="0 0 0"/>
-    </joint>
+    </joint> -->
     <link name="camera_link">
         <visual>
             <geometry>
-                <mesh filename="package://sayebot_description/meshes/camera.STL" scale="0.5 0.5 0.5"/>
-            </geometry>
-            <origin xyz="0 0 0" rpy="0 0 0"/>
+                <mesh filename="package://sayebot_description/meshes/camera.STL" scale="2.5 2.5 2.5"/>
+            </geometry>
+            <origin xyz="-0.15 0 -0.4" rpy="0 0 0"/>
         <material name="dark">
             <color rgba="0.8 0.8 0.8 1"></color>
@@ -203,5 +203,5 @@
         <parent link="base_link"/>
         <child link="camera_link"/>
-        <origin xyz="0.09 0 0.1" rpy="0 0 0"/>
+        <origin xyz="0.65 0 0.9" rpy="0 0 0"/>
     </joint>
 </robot>
